File: CAD/ecad/nucleo_shield_pcb.kicad_sch (KiCad schematic)
At the start: 12 parts, among them J1 CN7, J2 CN10, J3 Conn_01x02_Pin, J4 Conn_01x04_Socket, U1 ESP32-CAM, U2 ADXL345, U3 HC-SR04, U4 DM-OLED096-636

Commit message: Update KiCad schematic and layout with new ESP32 button circuitry
Parts:
- J3: footprint (none) -> Connector_PinHeader_2.54mm:PinHeader_1x02_P2.54mm_Vertical
- U1: footprint ESP32-CAM:ESP32-CAM -> components:ESP32-CAM
- U2: footprint SEN-09836:MODULE_SEN-09836 -> components:MODULE_SEN-09836
- U3: footprint HC-SR04:XCVR_HC-SR04 -> components:XCVR_HC-SR04
- U4: footprint DM-OLED096-636:MODULE_DM-OLED096-636 -> components:MODULE_DM-OLED096-636
Connections:
- net +3V3: now also U2.3 (CS)
- net GNDD: now also U2.6 (SDO)
- net SCL: now also J2.3 (Pin_3)
- net SDA: now also J2.5 (Pin_5)
- net at U3.2 (TRIG): now also J2.23 (Pin_23)
- net at U3.3 (ECHO): now also J2.19 (Pin_19)

Commit message: Fix component footprint libraries and resolve button shield pin mapping errors
Parts:
- removed H1: MountingHole, MountingHole:MountingHole_3.2mm_M3_ISO14580, symbol Mechanical:MountingHole
- added D2: 1N4148, Diode_THT:D_DO-35_SOD27_P7.62mm_Horizontal, symbol Diode:1N4148
- added SW1, SW2, SW3: CK_KMS2xxGP, Button_Switch_SMD:SW_SPST_PTS645Sx43SMTR92, symbol Switch:CK_KMS2xxGP
Connections:
- net GNDD: now also SW1.2, SW2.2, SW3.2
- net RESET: now also D2.1 (K), SW2.1
- net reset: now reaches U1.P$1 (GND@1)
- net reset: now also D2.2 (A)
- net at U1.P$13 (GPIO15): now also SW1.1
- net at J1.23 (Pin_23): now also SW3.1
Other:
- moved on the sheet: J1

Commit message: Update PCB and schematic: wire sensors, motor driver connector, and buttons
Parts:
- added J5: Conn_01x03_Pin, Connector_PinHeader_1.00mm:PinHeader_1x03_P1.00mm_Vertical, symbol Connector:Conn_01x03_Pin
- added J6: Conn_01x06_Pin, Connector_PinHeader_1.27mm:PinHeader_1x06_P1.27mm_Vertical, symbol Connector:Conn_01x06_Pin
- J1: value CN7 -> Conn_02x19_Odd_Even
Connections:
- net +5V: now also J5.3 (Pin_3)
- net E5V: now also J5.1 (Pin_1)
- net GNDD: now also J4.MP (5), J5.2 (Pin_2)
- net at J2.13 (Pin_13): now also J6.6 (Pin_6)
- net at J2.15 (Pin_15): now also J6.1 (Pin_1)
- net at J2.24 (Pin_24): now also J6.2 (Pin_2)
- net at J2.26 (Pin_26): now also J6.3 (Pin_3)
- net at J2.28 (Pin_28): now also J6.4 (Pin_4)
- net at J2.30 (Pin_30): now also J6.5 (Pin_5)
- no-connect marks 0 -> 52

Commit message: Configure 2.0mm JST PH connector for SGP30 sensor and generate Gerbers
Parts:
- J4: footprint Connector_JST:JST_ACH_BM04B-ACHSS-A-GAN-ETF_1x04-1MP_P1.20mm_Vertical -> Connector_JST:JST_PH_B4B-PH-K_1x04_P2.00mm_Vertical
Connections:
- net GNDD: no longer J4.MP (5)
Changed lines of the file:
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@@
 	(text "SGP30"
 		(exclude_from_sim no)
-		(at 69.088 126.238 0)
+		(at 84.582 117.094 0)
 		(effects
 			(font
@@
 	(symbol
 		(lib_id "power:GNDD")
-		(at 83.82 119.38 90)
-		(unit 1)
-		(body_style 1)
-		(exclude_from_sim no)
-		(in_bom yes)
-		(on_board yes)
-		(in_pos_files yes)
-		(dnp no)
-		(fields_autoplaced yes)
-		(property "Reference" "#PWR032"
-			(at 90.17 119.38 0)
-			(hide yes)
-			(show_name no)
-			(do_not_autoplace no)
-			(effects
-				(font
-					(size 1.27 1.27)
-				)
-			)
-		)
-		(property "Value" "GNDD"
-			(at 87.63 119.3801 90)
-			(show_name no)
-			(do_not_autoplace no)
-			(effects
-				(font
-					(size 1.27 1.27)
-				)
-				(justify right)
-			)
-		)
-		(property "Footprint" ""
-			(at 83.82 119.38 0)
-			(hide yes)
-			(show_name no)
-			(do_not_autoplace no)
-			(effects
-				(font
-					(size 1.27 1.27)
-				)
-			)
-		)
-		(property "Datasheet" ""
-			(at 83.82 119.38 0)
-			(hide yes)
-			(show_name no)
-			(do_not_autoplace no)
-			(effects
-				(font
-					(size 1.27 1.27)
-				)
-			)
-		)
-		(property "Description" "Power symbol creates a global label with name \"GNDD\" , digital ground"
-			(at 83.82 119.38 0)
-			(hide yes)
-			(show_name no)
-			(do_not_autoplace no)
-			(effects
-				(font
-					(size 1.27 1.27)
-				)
-			)
-		)
-		(pin "1"
-		)
-		(instances
-			(project "nucleo_shield_pcb"
-				(path "/9278c48a-e3d9-46fc-9342-1a833157c1d8"
-					(reference "#PWR032")
-					(unit 1)
-				)
-			)
-		)
-	)
-	(symbol
-		(lib_id "power:GNDD")
 		(at 118.11 161.29 180)
 		(unit 1)
@@
 		(fields_autoplaced yes)
 		(property "Reference" "J4"
-			(at 77.47 127.0001 0)
+			(at 79.375 116.84 0)
 			(show_name no)
 			(do_not_autoplace no)
@@
 					(size 1.27 1.27)
 				)
-				(justify left)
 			)
 		)
 		(property "Value" "Conn_01x04_Socket"
-			(at 77.47 124.4601 0)
+			(at 79.375 119.38 0)
 			(show_name no)
 			(do_not_autoplace no)
@@
 					(size 1.27 1.27)
 				)
-				(justify left)
 			)
 		)
-		(property "Footprint" "Connector_JST:JST_ACH_BM04B-ACHSS-A-GAN-ETF_1x04-1MP_P1.20mm_Vertical"
+		(property "Footprint" "Connector_JST:JST_PH_B4B-PH-K_1x04_P2.00mm_Vertical"
 			(at 78.74 127 0)
 			(hide yes)
@@
 		(pin "2"
 		)
-		(pin "MP"
-		)
 		(instances

Commit message: Updated Schematic, removed TODO
Other:
- note removed: "TODO"
Changed lines of the file:
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@@
 	(generator_version "10.0")
 	(paper "A4")
-	(text "TODO"
-		(exclude_from_sim no)
-		(at 105.41 81.026 0)
-		(effects
-			(font
-				(size 2.54 2.54)
-				(color 255 9 6 1)
-			)
-		)
-	)
 	(text "SGP30"
 		(exclude_from_sim no)
